File: h4k1/h4k1.brd (EAGLE design)
At the start: 250 x 80 mm, 190 parts, among them IC1 STM32F10XCXT6, J2 PJ-313D-AUDIO-JACK, J3 USB-AF10, K1 CHERRY-MX-LED, K10 CHERRY-MX-LED, K11 CHERRY-MX, K12 CHERRY-MX, K13 CHERRY-MX, K14 CHERRY-MX, K15 CHERRY-MX, K16 CHERRY-MX, K17 CHERRY-MX, K18 CHERRY-MX, K19 CHERRY-MX, K2 CHERRY-MX-LED, K20 CHERRY-MX-LED, K21 CHERRY-MX-LED, K22 CHERRY-MX-LED, K23 CHERRY-MX, K24 CHERRY-MX, K25 CHERRY-MX, K26 CHERRY-MX, K27 CHERRY-MX, K28 CHERRY-MX, K29 CHERRY-MX, K3 CHERRY-MX-LED, K30 CHERRY-MX, K31 CHERRY-MX, K32 CHERRY-MX, K33 CHERRY-MX-LED, K34 CHERRY-MX-LED, K35 CHERRY-MX-LED, K36 CHERRY-MX-LED, K37 CHERRY-MX-LED, K38 CHERRY-MX-LED, K39 CHERRY-MX-LED, K4 CHERRY-MX-LED, K40 CHERRY-MX-LED, K41 CHERRY-MX-LED, K42 CHERRY-MX-LED, K43 CHERRY-MX-LED, K44 CHERRY-MX-LED, K45 CHERRY-MX-LED, K46 CHERRY-MX-LED, K5 CHERRY-MX-LED, K6 CHERRY-MX-LED, K65 EVQPUL02K, K66 EVQPUL02K, K67 K3-1280S-F2, K7 CHERRY-MX-LED, K8 CHERRY-MX-LED, K9 CHERRY-MX-LED, U1 G850G, U3 PCM2704CDB, X4 12M

Commit message: re-layout keyboard switch
Parts:
- moved K46 228.5 mm to (239.0, 68.5)
- moved D9 228.3 mm to (8.72, 46.5)
- moved D46 225.1 mm to (236.4, 71.3), turned to 0 degrees
- moved K9 218.9 mm to (18.1, 30.5)
- moved D45 216.1 mm to (245.8, 80.6), turned to 0 degrees
- moved D10 198.2 mm to (39.1, 33.5), turned to 0 degrees
- moved K10 191.9 mm to (44.2, 30.5)
- moved K45 190.5 mm to (220.0, 68.5), turned to 0 degrees
- moved D47 184.9 mm to (-41.6, 70.5)
- moved D44 178.1 mm to (226.8, 80.6), turned to 0 degrees
- moved D40 155.9 mm to (249.9, -31.1)
- moved D11 155.7 mm to (60.4, 33.2), turned to 0 degrees
- moved K44 152.5 mm to (201.0, 68.5), turned to 0 degrees
- moved K11 151.5 mm to (63.2, 30.5)
- moved D43 140.3 mm to (207.7, 80.6), turned to 0 degrees
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Routing:
- net N$2: track 321.3 -> 0.00 mm, vias 6 -> 0
- net N$5: track 288.0 -> 0.00 mm, vias 7 -> 0
- net N$23: track 269.3 -> 0.00 mm, vias 10 -> 0
- net N$15: track 259.7 -> 0.00 mm, vias 8 -> 0
- net KB_R1: track 213.6 -> 0.00 mm
- net N$11: track 199.1 -> 0.00 mm, vias 7 -> 0
- net N$20: track 172.5 -> 0.00 mm, vias 6 -> 0
- net N$13: track 163.3 -> 0.00 mm, vias 6 -> 0
- net KB_R4: track 143.7 -> 0.00 mm
- net KB_R2: track 134.9 -> 0.00 mm
- net KB_R5: track 131.6 -> 0.00 mm
- net KB_R6: track 101.3 -> 0.00 mm
- net N$17: track 91.5 -> 0.00 mm, vias 4 -> 0
- net KB_R3: track 88.9 -> 0.00 mm
- net N$12: track 3.53 -> 0.00 mm
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Other:
- board size 250 x 80 mm -> 373.5 x 213 mm

Commit message: stm32 layout done
Parts:
- added R37, R38: 15, hqc:0805
- C1, C10, C11, C12, C13, C14, C15, C16, C17, C18, C19, C2, C3, C34, C35, C4, C7, C8, C9, L1, L2, R1, R10, R11, R12, R13, R14, R15, R16, R17, R18, R19, R2, R20, R21, R22, R23, R24, R25, R3, R35, R36, R4, R5, R6, R7, R8, R9: device hqc-basic:0603 -> hqc:0805
- C5, C6: value 4.7uF -> 15pF; device hqc-basic:0603 -> hqc:0805
- K10, K20, K21, K22, K34, K35, K38, K39, K41, K42, K43, K44, K45: value CHERRY-MX-LED -> CHERRY-MX; device hqc:CHERRY-MX-LED -> hqc:CHERRY-MX
- K17, K25: value CHERRY-MX -> CHERRY-MX-LED; device hqc:CHERRY-MX -> hqc:CHERRY-MX-LED
- moved U$4 432.0 mm to (125.0, 40.0), flipped to the bottom
- moved X2 298.2 mm to (112.1, 5.40), flipped to the bottom
- moved R17 290.6 mm to (121.3, 4.13), flipped to the bottom, turned to 90 degrees
- moved C2 285.2 mm to (121.9, 11.7), flipped to the bottom, turned to 270 degrees
- moved C3 285.2 mm to (116.5, 20.6), flipped to the bottom, turned to 180 degrees
- moved L1 284.8 mm to (101.0, 5.08), flipped to the bottom
- moved C6 284.8 mm to (117.2, 4.13), flipped to the bottom, turned to 90 degrees
- moved C5 284.5 mm to (119.1, 4.13), flipped to the bottom, turned to 90 degrees
- moved C9 284.2 mm to (106.0, 5.08), flipped to the bottom, turned to 180 degrees
- moved R18 283.2 mm to (101.0, 6.99), flipped to the bottom
- moved C8 282.6 mm to (106.0, 6.99), flipped to the bottom, turned to 180 degrees
- moved C7 281.3 mm to (106.0, 9.21), flipped to the bottom
- moved X1 277.2 mm to (118.1, 6.67), flipped to the bottom
- moved C4 273.7 mm to (104.1, 16.2), flipped to the bottom, turned to 90 degrees
- moved C1 271.1 mm to (106.4, 16.2), flipped to the bottom, turned to 90 degrees
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Connections:
- new net N$72: IC1.32, R37.P$1
- new net N$74: IC1.33, R38.P$1
- new net SWDCLK: IC1.37
- new net SWDIO: IC1.34
- net KB_C1: now also IC1.10
- net KB_C2: now also IC1.11
- net KB_C3: now also IC1.12
- net KB_C4: now also IC1.13
- net KB_C5: now also IC1.14
- net KB_C6: now also IC1.15
- net KB_C7: now also IC1.16
- net KB_C8: now also IC1.17
- net KB_R1: now also IC1.18
- net KB_R2: now also IC1.19
- net KB_R3: now also IC1.20
- net KB_R4: now also IC1.39
- net KB_R5: now also IC1.40
- net KB_R6: now also IC1.41
- net KB_R7: now also IC1.42
- net USB3+: now also R38.P$2
- net USB3-: now also R37.P$2
Routing:
- net N$11: track 0.00 -> 317.3 mm, vias 0 -> 10
- net N$2: track 0.00 -> 290.0 mm, vias 0 -> 5
- net N$23: track 0.00 -> 276.3 mm, vias 0 -> 13
- net N$13: track 0.00 -> 271.3 mm, vias 0 -> 12
- net KB_R1: track 0.00 -> 257.7 mm, vias 0 -> 2
- net N$15: track 0.00 -> 251.1 mm, vias 0 -> 10
- net N$5: track 0.00 -> 246.9 mm, vias 0 -> 9
- net N$20: track 0.00 -> 184.4 mm, vias 0 -> 5
- net KB_R2: track 0.00 -> 155.6 mm, vias 0 -> 1
- net KB_R5: track 0.00 -> 154.2 mm
- net N$17: track 0.00 -> 144.4 mm, vias 0 -> 8
- net KB_R4: track 0.00 -> 142.4 mm
- net KB_R3: track 0.00 -> 140.7 mm
- net KB_R6: track 0.00 -> 86.6 mm, vias 0 -> 1
- net GND: track 115.7 -> 176.8 mm, vias 6 -> 8
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Other:
- board size 373.5 x 213 mm -> 250 x 80 mm

Commit message: layout without led
Parts:
- removed D51, D52, D53, D54, D55, D56: (no value), hqc-basic:SOD-323
- moved K66 555.3 mm to (230.0, 72.2), flipped to the bottom, turned to 180 degrees
- moved K67 499.6 mm to (125.0, 76.1), flipped to the bottom
- moved R38 468.2 mm to (139.7, 14.2), flipped to the bottom, turned to 180 degrees
- moved R37 466.1 mm to (139.8, 16.4), flipped to the bottom, turned to 180 degrees
- moved R36 454.1 mm to (132.7, 39.4), flipped to the bottom, turned to 90 degrees
- moved R35 451.4 mm to (134.9, 39.3), flipped to the bottom, turned to 90 degrees
- moved C35 444.4 mm to (129.8, 39.4), flipped to the bottom, turned to 90 degrees
- moved C34 435.2 mm to (121.2, 40.0), flipped to the bottom, turned to 90 degrees
- moved K65 431.3 mm to (20.0, 72.2), flipped to the bottom, turned to 180 degrees
- moved R25 398.5 mm to (146.9, 4.06), flipped to the bottom, turned to 90 degrees
- moved R23 398.1 mm to (155.0, 4.06), flipped to the bottom, turned to 90 degrees
- moved R24 397.2 mm to (149.6, 4.06), flipped to the bottom, turned to 270 degrees
- moved C19 393.7 mm to (157.5, 4.06), flipped to the bottom, turned to 270 degrees
- moved R22 392.9 mm to (152.4, 4.06), flipped to the bottom, turned to 270 degrees
- moved C15 390.4 mm to (158.5, 17.7), flipped to the bottom
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Connections:
- removed net 3V3: C18.P$2, C19.P$2, L2.P$1, R22.P$2, U1.16, U1.24, U2.2
- removed net N$92: D53.P$2
- removed net N$93: D54.P$2
- removed net N$94: D55.P$2
- removed net N$95: D56.P$2
- net N$11: no longer D52.P$1
- net N$13: no longer D53.P$1
- net N$15: no longer D54.P$1
- net N$17: no longer D55.P$1
- net N$20: no longer D56.P$1
- net N$23: no longer D51.P$1
- net VDD: now also C18.P$2, C19.P$2, L2.P$1, R22.P$2, U1.16, U1.24, U2.2
Routing:
- net GND: track 176.8 -> 470.5 mm, vias 8 -> 29
- net KB_R7: track 0.00 -> 291.4 mm, vias 0 -> 3
- net VDD: track 42.8 -> 257.4 mm, vias 2 -> 7
- net USB1+: track 0.00 -> 185.1 mm, vias 0 -> 2
- net USB1-: track 0.00 -> 183.4 mm, vias 0 -> 2
- net 5V: track 0.00 -> 180.0 mm, vias 0 -> 6
- net N$20: track 184.4 -> 344.4 mm, vias 5 -> 9
- net HOST_USB-: track 0.00 -> 148.0 mm, vias 0 -> 1
- net HOST_USB+: track 0.00 -> 144.7 mm, vias 0 -> 1
- net USB2+: track 0.00 -> 138.4 mm, vias 0 -> 2
- net USB2-: track 0.00 -> 115.0 mm, vias 0 -> 4
- net KB_R6: track 86.6 -> 192.6 mm, vias 1 -> 4
- net N$17: track 144.4 -> 246.1 mm, vias 8 -> 10
- net N$5: track 246.9 -> 340.5 mm, vias 9 -> 11
- net N$2: track 290.0 -> 367.6 mm, vias 5 -> 11
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- removed copper zone on layer 1, net GND
- removed copper zone on layer 16, net GND
Other:
- outline, holes or cut-outs redrawn
