File: h4k1/h4k1.sch (EAGLE design)
At the start: 192 parts, among them IC1 STM32F10XCXT6, J2 PJ-313D-AUDIO-JACK, J3 USB-AF10, K1 CHERRY-MX-LED, K10 CHERRY-MX, K11 CHERRY-MX, K12 CHERRY-MX, K13 CHERRY-MX, K14 CHERRY-MX, K15 CHERRY-MX, K16 CHERRY-MX, K17 CHERRY-MX-LED, K18 CHERRY-MX, K19 CHERRY-MX, K2 CHERRY-MX-LED, K20 CHERRY-MX, K21 CHERRY-MX, K22 CHERRY-MX, K23 CHERRY-MX, K24 CHERRY-MX, K25 CHERRY-MX-LED, K26 CHERRY-MX, K27 CHERRY-MX, K28 CHERRY-MX, K29 CHERRY-MX, K3 CHERRY-MX-LED, K30 CHERRY-MX, K31 CHERRY-MX, K32 CHERRY-MX, K33 CHERRY-MX-LED, K34 CHERRY-MX, K35 CHERRY-MX, K36 CHERRY-MX-LED, K37 CHERRY-MX-LED, K38 CHERRY-MX, K39 CHERRY-MX, K4 CHERRY-MX-LED, K40 CHERRY-MX-LED, K41 CHERRY-MX, K42 CHERRY-MX, K43 CHERRY-MX, K44 CHERRY-MX, K45 CHERRY-MX, K46 CHERRY-MX-LED, K5 CHERRY-MX-LED, K6 CHERRY-MX-LED, K65 EVQPUL02K, K66 EVQPUL02K, K67 K3-1280S-F2, K7 CHERRY-MX-LED, K8 CHERRY-MX-LED, K9 CHERRY-MX-LED, U1 G850G, U3 PCM2704CDB, X4 12M

Commit message: layout without led
Parts:
- removed D51, D52, D53, D54, D55, D56: (no value), hqc-basic:IN4148WS-SWITCHING-DIODE
Connections:
- removed net 3V3: C18.P$2, C19.P$2, L2.P$1, R22.P$2, U1.DVDD, U1.V33, U2.VOUT
- removed net N$92: D53.P$2
- removed net N$93: D54.P$2
- removed net N$94: D55.P$2
- removed net N$95: D56.P$2
- net N$11: no longer D52.P$1
- net N$13: no longer D53.P$1
- net N$15: no longer D54.P$1
- net N$17: no longer D55.P$1
- net N$20: no longer D56.P$1
- net N$23: no longer D51.P$1
- net VDD: now also C18.P$2, C19.P$2, L2.P$1, R22.P$2, U1.DVDD, U1.V33, U2.VOUT
Changed lines of the file:
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@@
 <part name="D49" library="hqc-basic" deviceset="IN4148WS-SWITCHING-DIODE" device=""/>
 <part name="D50" library="hqc-basic" deviceset="IN4148WS-SWITCHING-DIODE" device=""/>
-<part name="D51" library="hqc-basic" deviceset="IN4148WS-SWITCHING-DIODE" device=""/>
-<part name="D52" library="hqc-basic" deviceset="IN4148WS-SWITCHING-DIODE" device=""/>
-<part name="D53" library="hqc-basic" deviceset="IN4148WS-SWITCHING-DIODE" device=""/>
-<part name="D54" library="hqc-basic" deviceset="IN4148WS-SWITCHING-DIODE" device=""/>
-<part name="D55" library="hqc-basic" deviceset="IN4148WS-SWITCHING-DIODE" device=""/>
-<part name="D56" library="hqc-basic" deviceset="IN4148WS-SWITCHING-DIODE" device=""/>
 <part name="R1" library="hqc" deviceset="R-0805" device="" value="10k"/>
 <part name="R2" library="hqc" deviceset="R-0805" device="" value="10k"/>
@@
 <part name="R37" library="hqc" deviceset="R-0805" device="" value="15"/>
 <part name="R38" library="hqc" deviceset="R-0805" device="" value="15"/>
+<part name="VDD16" library="supply1" deviceset="VDD" device=""/>
 </parts>
 <sheets>
@@
 <instance part="D49" gate="G$1" x="45.72" y="-307.34"/>
 <instance part="D50" gate="G$1" x="104.14" y="-307.34"/>
-<instance part="D51" gate="G$1" x="162.56" y="-307.34"/>
-<instance part="D52" gate="G$1" x="220.98" y="-307.34"/>
-<instance part="D53" gate="G$1" x="279.4" y="-307.34"/>
-<instance part="D54" gate="G$1" x="337.82" y="-307.34"/>
-<instance part="D55" gate="G$1" x="396.24" y="-307.34"/>
-<instance part="D56" gate="G$1" x="454.66" y="-307.34"/>
 <instance part="R1" gate="G$1" x="40.64" y="-83.82" rot="R90"/>
 <instance part="R2" gate="G$1" x="99.06" y="-83.82" rot="R90"/>
@@
 <instance part="R37" gate="G$1" x="30.48" y="38.1" rot="R180"/>
 <instance part="R38" gate="G$1" x="30.48" y="35.56" rot="R180"/>
+<instance part="VDD16" gate="G$1" x="73.66" y="256.54"/>
 </instances>
 <busses>
@@
 <wire x1="215.9" y1="-246.38" x2="215.9" y2="-276.86" width="0.1524" layer="91"/>
 <junction x="215.9" y="-246.38"/>
-<pinref part="D52" gate="G$1" pin="P$1"/>
 <wire x1="218.44" y1="-307.34" x2="215.9" y2="-307.34" width="0.1524" layer="91"/>
 <wire x1="215.9" y1="-276.86" x2="215.9" y2="-307.34" width="0.1524" layer="91"/>
@@
 <wire x1="274.32" y1="-246.38" x2="274.32" y2="-276.86" width="0.1524" layer="91"/>
 <junction x="274.32" y="-246.38"/>
-<pinref part="D53" gate="G$1" pin="P$1"/>
 <wire x1="276.86" y1="-307.34" x2="274.32" y2="-307.34" width="0.1524" layer="91"/>
 <wire x1="274.32" y1="-276.86" x2="274.32" y2="-307.34" width="0.1524" layer="91"/>
@@
 <wire x1="332.74" y1="-246.38" x2="332.74" y2="-276.86" width="0.1524" layer="91"/>
 <junction x="332.74" y="-246.38"/>
-<pinref part="D54" gate="G$1" pin="P$1"/>
 <wire x1="335.28" y1="-307.34" x2="332.74" y2="-307.34" width="0.1524" layer="91"/>
 <wire x1="332.74" y1="-276.86" x2="332.74" y2="-307.34" width="0.1524" layer="91"/>
@@
 <wire x1="391.16" y1="-246.38" x2="391.16" y2="-276.86" width="0.1524" layer="91"/>
 <junction x="391.16" y="-246.38"/>
-<pinref part="D55" gate="G$1" pin="P$1"/>
 <wire x1="393.7" y1="-307.34" x2="391.16" y2="-307.34" width="0.1524" layer="91"/>
 <wire x1="391.16" y1="-276.86" x2="391.16" y2="-307.34" width="0.1524" layer="91"/>
@@
 <wire x1="449.58" y1="-246.38" x2="449.58" y2="-276.86" width="0.1524" layer="91"/>
 <junction x="449.58" y="-246.38"/>
-<pinref part="D56" gate="G$1" pin="P$1"/>
 <wire x1="452.12" y1="-307.34" x2="449.58" y2="-307.34" width="0.1524" layer="91"/>
 <wire x1="449.58" y1="-276.86" x2="449.58" y2="-307.34" width="0.1524" layer="91"/>
@@
 <wire x1="157.48" y1="-276.86" x2="157.48" y2="-246.38" width="0.1524" layer="91"/>
 <junction x="157.48" y="-246.38"/>
-<pinref part="D51" gate="G$1" pin="P$1"/>
 <wire x1="160.02" y1="-307.34" x2="157.48" y2="-307.34" width="0.1524" layer="91"/>
 <wire x1="157.48" y1="-276.86" x2="157.48" y2="-307.34" width="0.1524" layer="91"/>
@@
 <pinref part="D48" gate="G$1" pin="P$2"/>
 <wire x1="459.74" y1="-276.86" x2="457.2" y2="-276.86" width="0.1524" layer="91"/>
-<wire x1="459.74" y1="-276.86" x2="459.74" y2="-271.78" width="0.1524" layer="91"/>
-<wire x1="459.74" y1="-271.78" x2="434.34" y2="-271.78" width="0.1524" layer="91"/>
-<wire x1="434.34" y1="-271.78" x2="434.34" y2="-281.94" width="0.1524" layer="91"/>
-<wire x1="434.34" y1="-281.94" x2="424.18" y2="-281.94" width="0.1524" layer="91"/>
+<wire x1="459.74" y1="-276.86" x2="459.74" y2="-281.94" width="0.1524" layer="91"/>
+<wire x1="459.74" y1="-281.94" x2="424.18" y2="-281.94" width="0.1524" layer="91"/>
 <pinref part="K67" gate="G$1" pin="P$3"/>
 </segment>
@@
 </segment>
 </net>
-<net name="N$92" class="0">
-<segment>
-<pinref part="D53" gate="G$1" pin="P$2"/>
-<wire x1="284.48" y1="-307.34" x2="281.94" y2="-307.34" width="0.1524" layer="91"/>
-</segment>
-</net>
-<net name="N$93" class="0">
-<segment>
-<pinref part="D54" gate="G$1" pin="P$2"/>
-<wire x1="342.9" y1="-307.34" x2="340.36" y2="-307.34" width="0.1524" layer="91"/>
-</segment>
-</net>
 <net name="N$94" class="0">
 <segment>
-<pinref part="D55" gate="G$1" pin="P$2"/>
 <wire x1="401.32" y1="-307.34" x2="398.78" y2="-307.34" width="0.1524" layer="91"/>
-</segment>
-</net>
-<net name="N$95" class="0">
-<segment>
-<pinref part="D56" gate="G$1" pin="P$2"/>
-<wire x1="459.74" y1="-307.34" x2="457.2" y2="-307.34" width="0.1524" layer="91"/>
 </segment>
 </net>
@@
 <pinref part="R35" gate="G$1" pin="P$2"/>
 <wire x1="309.88" y1="76.2" x2="309.88" y2="73.66" width="0.1524" layer="91"/>
+</segment>
+<segment>
+<pinref part="U2" gate="AMS1117-33" pin="VOUT"/>
+<wire x1="60.96" y1="251.46" x2="73.66" y2="251.46" width="0.1524" layer="91"/>
+<label x="66.04" y="251.46" size="1.778" layer="95"/>
+<pinref part="VDD16" gate="G$1" pin="VDD"/>
+<wire x1="73.66" y1="251.46" x2="73.66" y2="254" width="0.1524" layer="91"/>
+</segment>
+<segment>
+<pinref part="U1" gate="GL750G" pin="V33"/>
+<wire x1="76.2" y1="213.36" x2="86.36" y2="213.36" width="0.1524" layer="91"/>
+<label x="78.74" y="213.36" size="1.778" layer="95"/>
+</segment>
+<segment>
+<pinref part="L2" gate="G$1" pin="P$1"/>
+<wire x1="-45.72" y1="233.68" x2="-58.42" y2="233.68" width="0.1524" layer="91"/>
+<label x="-58.42" y="233.68" size="1.778" layer="95"/>
+</segment>
+<segment>
+<pinref part="U1" gate="GL750G" pin="DVDD"/>
+<wire x1="76.2" y1="193.04" x2="86.36" y2="193.04" width="0.1524" layer="91"/>
+<label x="78.74" y="193.04" size="1.778" layer="95"/>
+</segment>
+<segment>
+<wire x1="121.92" y1="190.5" x2="132.08" y2="190.5" width="0.1524" layer="91"/>
+<pinref part="C19" gate="G$1" pin="P$2"/>
+<wire x1="132.08" y1="190.5" x2="132.08" y2="187.96" width="0.1524" layer="91"/>
+<pinref part="C18" gate="G$1" pin="P$2"/>
+<wire x1="121.92" y1="190.5" x2="121.92" y2="187.96" width="0.1524" layer="91"/>
+<wire x1="132.08" y1="190.5" x2="139.7" y2="190.5" width="0.1524" layer="91"/>
+<junction x="132.08" y="190.5"/>
+<label x="132.08" y="190.5" size="1.778" layer="95"/>
+</segment>
+<segment>
+<pinref part="R22" gate="G$1" pin="P$2"/>
+<wire x1="93.98" y1="198.12" x2="104.14" y2="198.12" width="0.1524" layer="91"/>
+<label x="96.52" y="198.12" size="1.778" layer="95"/>
 </segment>
 </net>
@@
 </segment>
 </net>
-<net name="3V3" class="0">
-<segment>
-<pinref part="U2" gate="AMS1117-33" pin="VOUT"/>
-<wire x1="60.96" y1="251.46" x2="73.66" y2="251.46" width="0.1524" layer="91"/>
-<label x="66.04" y="251.46" size="1.778" layer="95"/>
-</segment>
-<segment>
-<pinref part="U1" gate="GL750G" pin="V33"/>
-<wire x1="76.2" y1="213.36" x2="86.36" y2="213.36" width="0.1524" layer="91"/>
-<label x="78.74" y="213.36" size="1.778" layer="95"/>
-</segment>
-<segment>
-<pinref part="L2" gate="G$1" pin="P$1"/>
-<wire x1="-45.72" y1="233.68" x2="-58.42" y2="233.68" width="0.1524" layer="91"/>
-<label x="-58.42" y="233.68" size="1.778" layer="95"/>
-</segment>
-<segment>
-<pinref part="U1" gate="GL750G" pin="DVDD"/>
-<wire x1="76.2" y1="193.04" x2="86.36" y2="193.04" width="0.1524" layer="91"/>
-<label x="78.74" y="193.04" size="1.778" layer="95"/>
-</segment>
-<segment>
-<wire x1="121.92" y1="190.5" x2="132.08" y2="190.5" width="0.1524" layer="91"/>
-<pinref part="C19" gate="G$1" pin="P$2"/>
-<wire x1="132.08" y1="190.5" x2="132.08" y2="187.96" width="0.1524" layer="91"/>
-<pinref part="C18" gate="G$1" pin="P$2"/>
-<wire x1="121.92" y1="190.5" x2="121.92" y2="187.96" width="0.1524" layer="91"/>
-<wire x1="132.08" y1="190.5" x2="139.7" y2="190.5" width="0.1524" layer="91"/>
-<junction x="132.08" y="190.5"/>
-<label x="132.08" y="190.5" size="1.778" layer="95"/>
-</segment>
-<segment>
-<pinref part="R22" gate="G$1" pin="P$2"/>
-<wire x1="93.98" y1="198.12" x2="104.14" y2="198.12" width="0.1524" layer="91"/>
-<label x="96.52" y="198.12" size="1.778" layer="95"/>
-</segment>
-</net>

Commit message: WIP: led layout
Parts:
- added R39, R40, R41, R42: 200, hqc:R-0805
- added T1: DBG, hqc-connector:CLIP-8P-1.27
Connections:
- removed net SWDCLK: IC1PORTA_H.PA14
- new net LED_C1: IC1PORTB_H.PB10, K1.LED+, K17.LED+, K25.LED+, K9.LED+
- new net LED_C2: IC1PORTB_H.PB11, K2.LED+, K3.LED+, K5.LED+, K6.LED+
- new net LED_C3: IC1PORTB_H.PB12, K4.LED+, K40.LED+, K7.LED+, K8.LED+
- new net LED_C4: IC1PORTB_H.PB13, K33.LED+, K36.LED+, K37.LED+, K46.LED+
- new net LED_R1: K25.LED-, K46.LED-, K6.LED-, K7.LED-, R39.P$2
- new net LED_R2: K17.LED-, K33.LED-, K5.LED-, K8.LED-, R40.P$2
- new net LED_R3: K3.LED-, K37.LED-, K4.LED-, K9.LED-, R41.P$2
- new net LED_R4: K1.LED-, K2.LED-, K36.LED-, K40.LED-, R42.P$2
- new net N$76: IC1PORTA_H.PA8, R39.P$1
- new net N$80: IC1PORTA_H.PA9, R40.P$1
- new net N$81: IC1PORTA_H.PA10, R41.P$1
- new net N$85: IC1PORTA_H.PA15, R42.P$1
- new net SWCLK: IC1PORTA_H.PA14, T1.7
- net GND: now also T1.8
- net SWDIO: now also T1.6
- net VDD: now also T1.5
Other:
- moved on the sheet: K1, K17, K2, K25, K3, K33, K36, K37, K4, K40, K46, K5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
